File: Isolated_FET_relay.sch (KiCad schematic (older format))
At the start: 20 parts, among them P1 CONN_01X05, P2 CONN_01X03, Q1 Q_NMOS_GDS, Q2 Q_NMOS_GDS, U1 Si8751, U2 REG113-XX-SOT23, U3 BGM111

Commit message: Created new layout concept
Connections:
- net V+: now also P2.3 (P3); no longer P2.1 (P1)
- net V-: now also P2.1 (P1); no longer P2.3 (P3)
Changed lines of the file:
@@
 F 3 "" H 10150 3775 50  0000 C CNN
 	1    10150 3775
-	1    0    0    -1
+	1    0    0    1
 $EndComp
 Text Label 2600 3350 0    60   ~ 0
